File: Hardware/Proiect_TSC.brd (EAGLE design)
At the start: 170.2 x 111.2 mm, 103 parts, among them IC1 BD5229G-TR, IC4 XC6220A331MR-G, J1 FH34SRJ-24S-0.5SH_99_, J2 SAMACSYS_PARTS_USB4110-GF-A, J3 QWIIC_RIGHT_ANGLE, J4 112A-TAAR-R03_ATTEND, Q1 SI1308EDL-T1-GE3, Q2 20V/4.2A/52mΩ/1.4W, Q3 20V/4.2A/52mΩ/1.4W, U1 W25Q512JVEIQ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

Commit message: Solved all open issues. Updated images and README.
Parts:
- D2: value ESP32_WROVER_AVX---SD0805S020S1R0_AVX_SD0805S020S1R0_0_0AVX_SD0805S020S1R0_0_0 -> SD0805S020S1R0
- R_CAPACITOR: value (none) -> 15
- SENSOR2: value ESP32_WROVER_BME680_BME680 -> BME688
- U: value ESP32_WROVER_SPARKFUN-IC-POWER_MCP73831 -> MCP73831
- moved TP4 119.5 mm to (146.3, 64.7)
- moved TP3 113.4 mm to (146.4, 60.6)
- moved TP5 110.3 mm to (88.7, 101.2)
- moved TP1 101.0 mm to (80.8, 101.1)
- moved TP2 100.6 mm to (73.1, 101.2)
- moved EPD_C5 25.7 mm to (116.9, 20.5)
- moved EPD_C6 21.6 mm to (111.3, 20.2)
- moved EPD_C7 18.1 mm to (106.3, 20.2)
- moved EPD_C8 14.8 mm to (101.5, 20.4)
- moved EPD_C9 11.1 mm to (96.3, 20.6)
- moved C7 10.7 mm to (90.4, 30.8)
- moved D4 9.20 mm to (83.2, 41.8)
- moved R9 9.07 mm to (68.2, 29.7)
- moved R6 8.45 mm to (39.1, 30.0)
- moved R_CL1 8.04 mm to (71.3, 29.9)
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Routing:
- net GND: track 730.5 -> 954.3 mm, vias 22 -> 52
- net 3V3: track 543.7 -> 447.4 mm
- net VBAT: track 118.4 -> 44.2 mm
- net N$13: track 6.91 -> 78.4 mm, vias 0 -> 6
- net RESE: track 35.1 -> 84.0 mm, vias 3 -> 0
- net N$6: track 30.0 -> 70.6 mm, vias 2 -> 4
- net VBUS: track 108.0 -> 146.4 mm
- net EPD_3V3: track 59.0 -> 89.0 mm
- net N$7: track 32.3 -> 61.2 mm, vias 2 -> 4
- net GPIO8: track 5.64 -> 32.6 mm, vias 2 -> 0
- net USB_D+: track 137.6 -> 164.4 mm
- net USB_D-: track 139.8 -> 165.3 mm
- net EPD_DC: track 104.4 -> 129.6 mm, vias 3 -> 6
- net N$10: track 9.20 -> 30.9 mm, vias 2 -> 4
- net SRC: track 46.6 -> 67.3 mm, vias 6 -> 5
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