File: Hardware/Proiect_TSC.sch (EAGLE design)
At the start: 103 parts, among them IC1 BD5229G-TR, IC4 XC6220A331MR-G, J1 FH34SRJ-24S-0.5SH_99_, J2 SAMACSYS_PARTS_USB4110-GF-A, J3 QWIIC_RIGHT_ANGLE, J4 112A-TAAR-R03_ATTEND, Q1 SI1308EDL-T1-GE3, Q2 20V/4.2A/52mΩ/1.4W, Q3 20V/4.2A/52mΩ/1.4W, U1 W25Q512JVEIQ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

Commit message: Solved all open issues. Updated images and README.
Parts:
- D2: value ESP32_WROVER_AVX---SD0805S020S1R0_AVX_SD0805S020S1R0_0_0AVX_SD0805S020S1R0_0_0 -> SD0805S020S1R0
- R_CAPACITOR: value (none) -> 15
- SENSOR2: value ESP32_WROVER_BME680_BME680 -> BME688
- U: value ESP32_WROVER_SPARKFUN-IC-POWER_MCP73831 -> MCP73831
Other:
- note added: "Battery Charge Level"
- note added: "DMG2305UX-7"
- note added: "Display Type Selector"
- note added: "E-Paper Display Header"
- note added: "E-Paper Drive Circuit"
- note added: "EPD Power"
- note added: "ESP32 C6"
- note added: "Environmental Sensor BME688"
- note added: "External NOR Flash 64MB"
- note added: "LDO Voltage Regulator"
- note added: "Li-Po Battery Charging Controller"
- note added: "Qwiic / Stemma QT"
- note added: "RTC Module DS3231SN"
- note added: "SD Card"
- note added: "SD0805S020S1R0"
- note added: "SPI ESD Protection Lines"
- note added: "Test Pads"
- note added: "USB C connector & ESD protection"
- note added: "Voltage Supervisor + Reset & Boot / IO Button"
- moved on the sheet: C1_BAT, C1_BAT1, C1_BAT2, C2_BAT, C3, C4, C4_USB, C5_USB, C7, C9, D1, D2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
